Commit message: update

File: install/servo_controller/share/servo_controller/urdf/my_turtlebot3_burger.urdf (robot description, URDF)
Before this commit: robot turtlebot_with_servo, 8 links, 7 joints
Links:
- added link servo_link_2, mass 0.01; collision cylinder length=0.1 radius=0.02; visual cylinder length=0.1 radius=0.02
- link base_link: geometry collision box size=0.2 0.2 0.1; visual box size=0.2 0.2 0.1
- link base_scan: geometry collision box size=0.05 0.05 0.1; visual box size=0.05 0.05 0.1
- link caster_back_link: geometry collision sphere radius=0.02
- link wheel_left_link: geometry collision cylinder length=0.02 radius=0.03; visual cylinder length=0.02 radius=0.03
- link wheel_right_link: geometry collision cylinder length=0.02 radius=0.03; visual cylinder length=0.02 radius=0.03
Joints:
- added joint servo_joint_2: type revolute, parent base_link, child servo_link_2, origin xyz=0 0 0.2 rpy=0 0 0, axis 0 1 0, limit lower=0 upper=1.57 effort=1.0 velocity=1.0
